Commit message: run successfully without imu
Signed-off-by: Hao Liang <hao.liang@shmastermatrix.com>

File: cartographer_ros/urdf/quanergy_2d.urdf (robot description, URDF)
Before this commit: robot cartographer_iCrane_2d, 2 links, 1 joints
Links:
- removed link base_link
Joints:
- removed joint Sensor_joint

Commit message: create base_link and sensor rviz model
Signed-off-by: Hao Liang <hao.liang@shmastermatrix.com>

File: cartographer_ros/urdf/quanergy_2d.urdf (robot description, URDF)
Before this commit: robot cartographer_iCrane_2d, 1 links, 0 joints
Links:
- added link base_link; visual box size=0.5 0.5 0.5
- link Sensor: geometry visual cylinder length=0.1 radius=0.06
Joints:
- added joint Sensor_joint: type fixed, parent base_link, child Sensor, origin xyz=0 0 0 rpy=0.0 0.0 0.0

Commit message: perfect urdf model
Signed-off-by: Hao Liang <hao.liang@shmastermatrix.com>

File: cartographer_ros/urdf/quanergy_2d.urdf (robot description, URDF)
Before this commit: robot cartographer_iCrane_2d, 2 links, 1 joints
Links:
- link Sensor: geometry visual cylinder length=0.11 radius=0.055
- link base_link: geometry visual box size=0.5 0.392 0.60
